File: KiCad/SFH203_photodetector.kicad_sch (KiCad schematic)
At the start: 19 parts, among them J1 V- GND V+, J4 Signal out, U1 ADA4898-2, U2 LT3032-12

Commit message: Update to KiCad7
Parts:
- J4: footprint Connector_Coaxial:SMA_Molex_73251-2120_EdgeMount_Horizontal -> custom:SMA_Molex_73251-2120_EdgeMount_Horizontal_mod
- LOGO1: Config DNF -> (none)
